File: kicad test/JTAG.kicad_sch (KiCad schematic)
At the start: 0 parts

Commit message: docs: modify mpu sch
Parts:
- added U1: 4001, symbol 4xxx:4001
Connections:
- new net: U1.10, U1.11
- new net: U1.12, U1.8
- new net: U1.13, U1.9
